Commit message: pushing bc pc is going into repair

File: src/simulation/urdf/components/left_drive.xacro (robot description, xacro)
@@ -1,5 +1,5 @@
 <?xml version="1.0"?>
 <robot xmlns:xacro="http://www.ros.org/wiki/xacro">
-    <xacro:macro name = "right_drive">
+    <xacro:macro name = "left_drive">
         <!-- Imports -->
          <!-- I dont understand why but ROS1 imports only work for imports T_T -->
@@ -10,15 +10,15 @@
         <!--     RIGHT CHASIS     -->
         <!-- =====================-->
-        <xacro:property name="rc_pos_x" value = "0.292"/>
-        <xacro:property name="rc_pos_y" value = "-0.115"/>
-        <xacro:property name="rc_pos_z" value = "-0.0125"/>
-        <xacro:property name="rc_col_x" value = "0.044"/>
-        <xacro:property name="rc_col_y" value = "1.1"/>
-        <xacro:property name="rc_col_z" value = "0.25"/>
-        <link name = "right_chasis">
+        <xacro:property name="lc_pos_x" value = "0.292"/>
+        <xacro:property name="lc_pos_y" value = "-0.115"/>
+        <xacro:property name="lc_pos_z" value = "-0.0125"/>
+        <xacro:property name="lc_col_x" value = "0.044"/>
+        <xacro:property name="lc_col_y" value = "1.1"/>
+        <xacro:property name="lc_col_z" value = "0.25"/>
+        <link name = "left_chasis">
             <!-- Inertial Values-->
             <inertial>
                 <mass value="6.019"/>
-                <origin xyz = "${rc_pos_x} ${rc_pos_y} ${rc_pos_z}"/>
+                <origin xyz = "${lc_pos_x} ${lc_pos_y} ${lc_pos_z}"/>
                 <inertia
                     ixx="0.919"
@@ -30,17 +30,17 @@
             </inertial>
             <!-- Visuals -->
-            <visual name = "rd_chasis_visual">
+            <visual name = "ld_chasis_visual">
                 <geometry>
                     <!-- And ros2 imports only work for meshes T_T -->
                     <mesh filename = "package://simulation/meshes/rd_chasis.stl"/>
                 </geometry>
-                <xacro:body_mat link_name = "rd_chasis"/>
+                <xacro:body_mat link_name = "ld_chasis"/>
             </visual>
             <!-- Collisions-->
-            <collision name = "rd_chasis_collision">
-                <geometry>
-                    <box size="${rc_col_x} ${rc_col_y} ${rc_col_z}"/>
-                </geometry>
-                <origin xyz="${rc_pos_x} ${rc_pos_y} ${rc_pos_z}" rpy="0 0 0"/>
+            <collision name = "ld_chasis_collision">
+                <geometry>
+                    <box size="${lc_col_x} ${lc_col_y} ${lc_col_z}"/>
+                </geometry>
+                <origin xyz="${lc_pos_x} ${lc_pos_y} ${lc_pos_z}" rpy="0 0 0"/>
             </collision>
         </link>
@@ -48,8 +48,8 @@
         <!--     BACK SWIVEL      -->
         <!-- =====================-->
-        <xacro:property name="bs_pos_x" value = "0.292"/>
-        <xacro:property name="bs_pos_y" value = "0.343"/>
-        <xacro:property name="bs_pos_z" value = "-0.211"/>
-        <link name = "back_swivel">
+        <xacro:property name="left_bs_pos_x" value = "0.292"/>
+        <xacro:property name="left_bs_pos_y" value = "0.343"/>
+        <xacro:property name="left_bs_pos_z" value = "-0.211"/>
+        <link name = "ld_back_swivel">
             <inertial>
                 <mass value="0.227"/>
@@ -65,17 +65,17 @@
             </inertial>
             <!-- Visuals -->
-            <visual name = "rd_back_swivel_visual">
-                <origin xyz="${-bs_pos_x} ${-bs_pos_y} ${-bs_pos_z}" rpy="0 0 0"/>
+            <visual name = "ld_back_swivel_visual">
+                <origin xyz="${-left_bs_pos_x} ${-left_bs_pos_y} ${-left_bs_pos_z}" rpy="0 0 0"/>
                 <geometry>
                     <!-- And ros2 imports only work for meshes T_T -->
                     <mesh filename = "package://simulation/meshes/rd_back_swivel.stl"/>
                 </geometry>
-                <xacro:body_mat link_name = "rd_back_swivel"/>
-            </visual>
-        </link>
-        <joint name="rd_to_bw" type="continuous">
-            <parent link="right_chasis"/>
-            <child link="back_swivel"/>
-            <origin xyz="${bs_pos_x} ${bs_pos_y} ${bs_pos_z}" rpy="0 0 0"/>
+                <xacro:body_mat link_name = "ld_back_swivel"/>
+            </visual>
+        </link>
+        <joint name="ld_to_bw" type="continuous">
+            <parent link="left_chasis"/>
+            <child link="ld_back_swivel"/>
+            <origin xyz="${left_bs_pos_x} ${left_bs_pos_y} ${left_bs_pos_z}" rpy="0 0 0"/>
             <axis xyz = "0 0 1"/>
         </joint>
@@ -83,8 +83,8 @@
         <!--     FRONT SWIVEL      -->
         <!-- =====================-->
-        <xacro:property name="fs_pos_x" value = "0.292"/>
-        <xacro:property name="fs_pos_y" value = "-0.574"/>
-        <xacro:property name="fs_pos_z" value = "-0.211"/>
-        <link name = "front_swivel">
+        <xacro:property name="ld_fs_pos_x" value = "0.292"/>
+        <xacro:property name="ld_fs_pos_y" value = "-0.574"/>
+        <xacro:property name="ld_fs_pos_z" value = "-0.211"/>
+        <link name = "ld_front_swivel">
             <inertial>
                 <mass value="0.227"/>
@@ -101,16 +101,16 @@
             <!-- Visuals -->
             <visual name = "rd_back_swivel_visual">
-                <origin xyz="${-fs_pos_x} ${-fs_pos_y} ${-fs_pos_z}" rpy="0 0 0"/>
+                <origin xyz="${-ld_fs_pos_x} ${-ld_fs_pos_y} ${-ld_fs_pos_z}" rpy="0 0 0"/>
                 <geometry>
                     <!-- And ros2 imports only work for meshes T_T -->
                     <mesh filename = "package://simulation/meshes/rd_front_swivel.stl"/>
                 </geometry>
-                <xacro:body_mat link_name = "rd_back_swivel"/>
+                <xacro:body_mat link_name = "ld_back_swivel"/>
             </visual>
         </link>
         <joint name="rd_to_fw" type="continuous">
-            <parent link="right_chasis"/>
-            <child link="front_swivel"/>
-            <origin xyz="${fs_pos_x} ${fs_pos_y} ${fs_pos_z}" rpy="0 0 0"/>
+            <parent link="left_chasis"/>
+            <child link="ld_front_swivel"/>
+            <origin xyz="${ld_fs_pos_x} ${ld_fs_pos_y} ${ld_fs_pos_z}" rpy="0 0 0"/>
             <axis xyz = "0 0 1"/>
         </joint>
@@ -118,8 +118,8 @@
         <!--     FRONT WHEEL      -->
         <!-- =====================-->
-        <xacro:property name="fw_pos_x" value = "0.292"/>
-        <xacro:property name="fw_pos_y" value = "-.574"/>
-        <xacro:property name="fw_pos_z" value = "-0.25"/>
-        <link name = "front_wheel">
+        <xacro:property name="ld_fw_pos_x" value = "0.292"/>
+        <xacro:property name="ld_fw_pos_y" value = "-.574"/>
+        <xacro:property name="ld_fw_pos_z" value = "-0.25"/>
+        <link name = "ld_front_wheel">
             <inertial>
                 <origin xyz = "0 0 0"/>
@@ -134,13 +134,13 @@
             </inertial>
             <!-- Visuals -->
-            <visual name = "rd_front_wheel_visual">
-                <origin xyz="${-fw_pos_x} ${-fw_pos_y} ${-fw_pos_z}" rpy="0 0 0"/>
+            <visual name = "ld_front_wheel_visual">
+                <origin xyz="${-ld_fw_pos_x} ${-ld_fw_pos_y} ${-ld_fw_pos_z}" rpy="0 0 0"/>
                 <geometry>
                     <!-- And ros2 imports only work for meshes T_T -->
                     <mesh filename = "package://simulation/meshes/rd_front_wheel.stl"/>
                 </geometry>
-                <xacro:body_mat link_name = "rw_back_swivel"/>
-            </visual>
-            <collision name = "rd_front_wheel_collision">
+                <xacro:body_mat link_name = "ld_back_swivel"/>
+            </visual>
+            <collision name = "ld_front_wheel_collision">
                 <origin xyz="0 0 0" rpy = "-1.5707 0 0"/>
                 <geometry>
@@ -152,9 +152,9 @@
             </collision>
         </link>
-        <joint name = "fw_to_fs" type = "continuous">
-            <parent link = "front_swivel"/>
-            <child link = "front_wheel"/>
+        <joint name = "ld_fw_to_fs" type = "continuous">
+            <parent link = "ld_front_swivel"/>
+            <child link = "ld_front_wheel"/>
             <!-- I dont understand why mathematically this works T_T-->
-            <origin xyz="${fw_pos_x - fs_pos_x} ${fw_pos_y - fs_pos_y} ${fw_pos_z - fs_pos_z}" rpy="0 0 0"/>
+            <origin xyz="${ld_fw_pos_x - ld_fs_pos_x} ${ld_fw_pos_y - ld_fs_pos_y} ${ld_fw_pos_z - ld_fs_pos_z}" rpy="0 0 0"/>
             <axis xyz = "0 1 0"/>
         </joint>
@@ -162,8 +162,8 @@
         <!--     BACK WHEEL       -->
         <!-- =====================-->
-        <xacro:property name="bw_pos_x" value = "0.292"/>
-        <xacro:property name="bw_pos_y" value = ".344"/>
-        <xacro:property name="bw_pos_z" value = "-0.25"/>
-        <link name = "back_wheel">
+        <xacro:property name="ld_bw_pos_x" value = "0.292"/>
+        <xacro:property name="ld_bw_pos_y" value = ".344"/>
+        <xacro:property name="ld_bw_pos_z" value = "-0.25"/>
+        <link name = "ld_back_wheel">
             <inertial>
                 <origin xyz = "0 0 0"/>
@@ -178,13 +178,13 @@
             </inertial>
             <!-- Visuals -->
-            <visual name = "rd_back_wheel_visual">
-                <origin xyz="${-bw_pos_x} ${-bw_pos_y} ${-bw_pos_z}" rpy="0 0 0"/>
+            <visual name = "ld_back_wheel_visual">
+                <origin xyz="${-ld_bw_pos_x} ${-ld_bw_pos_y} ${-ld_bw_pos_z}" rpy="0 0 0"/>
                 <geometry>
                     <!-- And ros2 imports only work for meshes T_T -->
                     <mesh filename = "package://simulation/meshes/rd_back_wheel.stl"/>
                 </geometry>
-                <xacro:body_mat link_name = "rw_back_swivel"/>
-            </visual>
-            <collision name = "rd_back_wheel_collision">
+                <xacro:body_mat link_name = "ld_back_swivel"/>
+            </visual>
+            <collision name = "ld_back_wheel_collision">
                 <origin xyz="0 0 0" rpy = "-1.5707 0 0"/>
                 <geometry>
@@ -196,9 +196,9 @@
             </collision>
         </link>
-        <joint name = "bw_to_bs" type = "continuous">
-            <parent link = "back_swivel"/>
-            <child link = "back_wheel"/>
+        <joint name = "ld_bw_to_bs" type = "continuous">
+            <parent link = "ld_back_swivel"/>
+            <child link = "ld_back_wheel"/>
             <!-- I dont understand why mathematically this works T_T-->
-            <origin xyz="${bw_pos_x - bs_pos_x} ${bw_pos_y - bs_pos_y} ${bw_pos_z - bs_pos_z}" rpy="0 0 0"/>
+            <origin xyz="${ld_bw_pos_x - left_bs_pos_x} ${ld_bw_pos_y - left_bs_pos_y} ${ld_bw_pos_z - left_bs_pos_z}" rpy="0 0 0"/>
             <axis xyz = "0 1 0"/>
         </joint>
